File: reference/hardware/Speedy MAP/Hardware/SpeedyMAP.kicad_pcb (KiCad board)
At the start: 2 copper layers, 16.5 x 57.2 mm, 27 parts, among them IC1 ATMEGA328-A, SW1 SW_SPST, U1 MPX4250, U2 MPX4250, U3 MPX4250, U4 MPX4250, U5 MCP4921-E/SN, Y1 Crystal

Commit message: Mostly complete SpeedyMAP firmware
Parts:
- moved U4 102.4 mm to (62.8, 84.6)
- moved C12 102.4 mm to (69.2, 73.2)
- moved C4 102.4 mm to (69.2, 80.8)
- moved C8 102.4 mm to (69.2, 77.0)
- moved R4 102.4 mm to (69.2, 84.6)
- moved U3 101.6 mm to (62.8, 119.8)
- moved C11 101.6 mm to (69.2, 108.4)
- moved C3 101.6 mm to (69.2, 116.0)
- moved C7 101.6 mm to (69.2, 112.2)
- moved R3 101.6 mm to (69.2, 119.8)
- moved IC1 90.4 mm to (95.2, 93.2)
- moved U5 90.4 mm to (78.0, 94.0)
- moved U1 86.6 mm to (117.0, 71.8)
- moved C9 86.6 mm to (108.0, 84.0)
- moved C1 86.5 mm to (108.0, 80.5)
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Routing:
- net GND: vias 1 -> 0
Other:
- board size 16.5 x 57.2 mm -> 100 x 100 mm
Changed lines of the file:
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@@
     (links 60)
     (no_connects 60)
-    (area 228.524999 81.204999 245.185001 138.505001)
+    (area 39.924999 39.924999 140.075001 140.075001)
     (thickness 1.6)
-    (drawings 13)
-    (tracks 1)
+    (drawings 8)
+    (tracks 0)
     (zones 0)
     (modules 27)
@@
   )
   (module Capacitors_SMD:C_0805_HandSoldering (layer F.Cu)
-    (at 193.04 96.52)
+    (at 108.04 80.52)
     (descr "Capacitor SMD 0805, hand soldering")
     (tags "capacitor 0805")
@@
   )
   (module Capacitors_SMD:C_0805_HandSoldering (layer F.Cu)
-    (at 193.04 121.92)
+    (at 108.04 110.92)
     (descr "Capacitor SMD 0805, hand soldering")
     (tags "capacitor 0805")
@@
   )
   (module Capacitors_SMD:C_0805_HandSoldering (layer F.Cu)
-    (at 170.18 127)
+    (at 69.18 116)
     (descr "Capacitor SMD 0805, hand soldering")
     (tags "capacitor 0805")
@@
   )
   (module Capacitors_SMD:C_0805_HandSoldering (layer F.Cu)
-    (at 170.18 97.79)
+    (at 69.18 80.79)
     (descr "Capacitor SMD 0805, hand soldering")
     (tags "capacitor 0805")
@@
   )
   (module Capacitors_SMD:C_0805_HandSoldering (layer F.Cu)
-    (at 193.04 92.71)
+    (at 108.04 76.71)
     (descr "Capacitor SMD 0805, hand soldering")
     (tags "capacitor 0805")
@@
   )
   (module Capacitors_SMD:C_0805_HandSoldering (layer F.Cu)
-    (at 193.04 125.73)
+    (at 108.04 114.73)
     (descr "Capacitor SMD 0805, hand soldering")
     (tags "capacitor 0805")
@@
   )
   (module Capacitors_SMD:C_0805_HandSoldering (layer F.Cu)
-    (at 170.18 123.19)
+    (at 69.18 112.19)
     (descr "Capacitor SMD 0805, hand soldering")
     (tags "capacitor 0805")
@@
   )
   (module Capacitors_SMD:C_0805_HandSoldering (layer F.Cu)
-    (at 170.18 93.98)
+    (at 69.18 76.98)
     (descr "Capacitor SMD 0805, hand soldering")
     (tags "capacitor 0805")
@@
   )
   (module Capacitors_SMD:C_0805_HandSoldering (layer F.Cu)
-    (at 193.04 100.33)
+    (at 108 84)
     (descr "Capacitor SMD 0805, hand soldering")
     (tags "capacitor 0805")
@@
   )
   (module Capacitors_SMD:C_0805_HandSoldering (layer F.Cu)
-    (at 193.04 129.54)
+    (at 108.04 118.54)
     (descr "Capacitor SMD 0805, hand soldering")
     (tags "capacitor 0805")
@@
   )
   (module Capacitors_SMD:C_0805_HandSoldering (layer F.Cu)
-    (at 170.18 119.38)
+    (at 69.18 108.38)
     (descr "Capacitor SMD 0805, hand soldering")
     (tags "capacitor 0805")
@@
   )
   (module Capacitors_SMD:C_0805_HandSoldering (layer F.Cu)
-    (at 170.18 90.17)
+    (at 69.18 73.17)
     (descr "Capacitor SMD 0805, hand soldering")
     (tags "capacitor 0805")
@@
   )
   (module Housings_QFP:TQFP-32_7x7mm_Pitch0.8mm (layer F.Cu)
-    (at 184.15 109.22)
+    (at 95.15 93.22)
     (descr "32-Lead Plastic Thin Quad Flatpack (PT) - 7x7x1.0 mm Body, 2.00 mm [TQFP] (see Microchip Packaging Specification 00000049BS.pdf)")
     (tags "QFP 0.8")
@@
   )
   (module Resistors_SMD:R_0805_HandSoldering (layer F.Cu)
-    (at 193.04 88.9)
+    (at 108.04 72.9)
     (descr "Resistor SMD 0805, hand soldering")
     (tags "resistor 0805")
@@
   )
   (module Resistors_SMD:R_0805_HandSoldering (layer F.Cu)
-    (at 193.04 118.11)
+    (at 108.04 107.11)
     (descr "Resistor SMD 0805, hand soldering")
     (tags "resistor 0805")
@@
   )
   (module Resistors_SMD:R_0805_HandSoldering (layer F.Cu)
-    (at 170.18 130.81)
+    (at 69.18 119.81)
     (descr "Resistor SMD 0805, hand soldering")
     (tags "resistor 0805")
@@
   )
   (module Resistors_SMD:R_0805_HandSoldering (layer F.Cu)
-    (at 170.18 101.6)
+    (at 69.18 84.6)
     (descr "Resistor SMD 0805, hand soldering")
     (tags "resistor 0805")
@@
   )
   (module MPX4250:MPX4250 (layer F.Cu)
-    (at 201.93 88.9 270)
+    (at 117 71.84 270)
     (fp_text reference U1 (at 2.54 2.54 270) (layer F.SilkS)
       (effects (font (size 1 1) (thickness 0.15)))
@@
   )
   (module MPX4250:MPX4250 (layer F.Cu)
-    (at 201.93 118.11 270)
+    (at 116.93 107.11 270)
     (fp_text reference U2 (at 2.54 2.54 270) (layer F.SilkS)
       (effects (font (size 1 1) (thickness 0.15)))
@@
   )
   (module MPX4250:MPX4250 (layer F.Cu)
-    (at 163.83 130.81 90)
+    (at 62.83 119.81 90)
     (fp_text reference U3 (at 2.54 2.54 90) (layer F.SilkS)
       (effects (font (size 1 1) (thickness 0.15)))
@@
   )
   (module MPX4250:MPX4250 (layer F.Cu)
-    (at 163.83 101.6 90)
+    (at 62.83 84.6 90)
     (fp_text reference U4 (at 2.54 2.54 90) (layer F.SilkS)
       (effects (font (size 1 1) (thickness 0.15)))
@@
   )
   (module Capacitors_SMD:C_0805_HandSoldering (layer F.Cu)
-    (at 240 134)
+    (at 182 128)
     (descr "Capacitor SMD 0805, hand soldering")
     (tags "capacitor 0805")
@@
   )
   (module Buttons_Switches_ThroughHole:SW_TH_Tactile_Omron_B3F-10xx (layer F.Cu)
-    (at 200.66 107.95)
+    (at 115.66 96.95)
     (descr SW_TH_Tactile_Omron_B3F-10xx)
     (tags "Omron B3F-10xx")
@@
   )
   (module Housings_SOIC:SOIC-8_3.9x4.9mm_Pitch1.27mm (layer F.Cu)
-    (at 167 110)
+    (at 78 94)
     (descr "8-Lead Plastic Small Outline (SN) - Narrow, 3.90 mm Body [SOIC] (see Microchip Packaging Specification 00000049BS.pdf)")
     (tags "SOIC 1.27")
@@
     )
   )
-  (gr_text "Flat side up" (at 151.13 124.46) (layer F.SilkS)
+  (gr_line (start 40 140) (end 40 40) (layer Edge.Cuts) (width 0.15))
+  (gr_line (start 140 140) (end 40 140) (layer Edge.Cuts) (width 0.15))
+  (gr_line (start 140 40) (end 140 140) (layer Edge.Cuts) (width 0.15))
+  (gr_line (start 40 40) (end 140 40) (layer Edge.Cuts) (width 0.15))
+  (gr_text "Flat side up" (at 50.13 113.46) (layer F.SilkS)
     (effects (font (size 1.5 1.5) (thickness 0.3)))
   )
-  (gr_text "Flat side up" (at 151.13 95.25) (layer F.SilkS)
+  (gr_text "Flat side up" (at 50.13 78.25) (layer F.SilkS)
     (effects (font (size 1.5 1.5) (thickness 0.3)))
   )
-  (gr_text "Flat side up" (at 214.63 95.25) (layer F.SilkS)
+  (gr_text "Flat side up" (at 129.63 79.25) (layer F.SilkS)
     (effects (font (size 1.5 1.5) (thickness 0.3)))
   )
-  (gr_text "Flat side up" (at 214.63 124.46) (layer F.SilkS)
+  (gr_text "Flat side up" (at 129.63 113.46) (layer F.SilkS)
     (effects (font (size 1.5 1.5) (thickness 0.3)))
   )
-  (gr_line (start 231.14 138.43) (end 242.57 138.43) (angle 90) (layer Edge.Cuts) (width 0.15))
-  (gr_line (start 231.14 81.28) (end 242.57 81.28) (angle 90) (layer Edge.Cuts) (width 0.15))
-  (gr_line (start 228.6 83.82) (end 228.6 135.89) (angle 90) (layer Edge.Cuts) (width 0.15))
-  (gr_arc (start 231.14 83.82) (end 228.6 83.82) (angle 90) (layer Edge.Cuts) (width 0.15))
-  (gr_arc (start 231.14 135.89) (end 231.14 138.43) (angle 90) (layer Edge.Cuts) (width 0.15))
-  (gr_line (start 245.11 83.82) (end 245.11 135.89) (angle 90) (layer Edge.Cuts) (width 0.15))
-  (gr_arc (start 242.57 135.89) (end 245.11 135.89) (angle 90) (layer Edge.Cuts) (width 0.15))
-  (gr_circle (center 241.3 86.36) (end 240.03 86.36) (layer Edge.Cuts) (width 0.15))
-  (gr_arc (start 242.57 83.82) (end 242.57 81.28) (angle 90) (layer Edge.Cuts) (width 0.15))
-  (via (at 236 130) (size 0.6) (drill 0.4) (layers F.Cu B.Cu) (net 2))
   (zone (net 2) (net_name GND) (layer F.Cu) (hatch edge 0.508)
-    (priority 1)
     (connect_pads (clearance 0.508))
     (min_thickness 0.254)
-    (fill yes (arc_segments 16) (thermal_gap 0.508) (thermal_bridge_width 0.508))
+    (fill (arc_segments 16) (thermal_gap 0.508) (thermal_bridge_width 0.508))
     (polygon
       (pts
-        (xy 244 137) (xy 230 137) (xy 230 83) (xy 244 83)
+        (xy 139 137) (xy 41 137) (xy 41 43) (xy 139 43)
       )
     )
@@
     (connect_pads (clearance 0.508))
     (min_thickness 0.254)
-    (fill yes (arc_segments 16) (thermal_gap 0.508) (thermal_bridge_width 0.508))
+    (fill (arc_segments 16) (thermal_gap 0.508) (thermal_bridge_width 0.508))
     (polygon
       (pts
-        (xy 244 137) (xy 230 137) (xy 230 83) (xy 244 83)
+        (xy 41 137) (xy 41 43) (xy 139 43) (xy 139 137)
       )
     )
